File: KiCad/Target_Master/Target.kicad_sch (KiCad schematic)
At the start: 0 parts

Commit message: Master board silkscreen and gerber files
Other:
- title: Laser Shooting Game Target Master -> Laser Arcade Master
Changed lines of the file:
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@@
 	(paper "A")
 	(title_block
-		(title "Laser Shooting Game Target Master")
-		(date "2025-04-04")
+		(title "Laser Arcade Master")
+		(date "2025-04-17")
 		(rev "A")
 		(company "Idaho State University")
