File: KiCad/Target_Master/UART.kicad_sch (KiCad schematic)
At the start: 13 parts, among them J3 USB_B_Mini, U3 FT232RL

Commit message: Finalized schematics
Parts:
- removed C9: 4.7uF, symbol Device:C_Polarized_Small_US
- added C1: 0.1uF, symbol Device:C_Small
- added C2: 4.7uF, symbol Device:C_Small
Connections:
- net +5V: now also C2.1
- net GND: now also C1.1, C2.2; no longer J3.4 (ID)
- net at U3.17 (3V3OUT): now also C1.2
Other:
- moved on the sheet: D3, D4

Commit message: Master PCB design, Slave board logos
Parts:
- added TP1, TP2, TP3, TP4: ~, 0_AKeller_Footprints:1x1_100mil_Header, symbol 0_AKeller_Parts:Test_Point
- C10: renamed from C7; footprint (none) -> Capacitor_SMD:C_0805_2012Metric_Pad1.18x1.45mm_HandSolder
- C11: renamed from C8; footprint (none) -> Capacitor_SMD:C_0805_2012Metric_Pad1.18x1.45mm_HandSolder
- C12: renamed from C2; footprint (none) -> Capacitor_SMD:C_0805_2012Metric_Pad1.18x1.45mm_HandSolder
- C13: renamed from C10; footprint (none) -> Capacitor_SMD:C_0805_2012Metric_Pad1.18x1.45mm_HandSolder
- C8: renamed from C1; footprint (none) -> Capacitor_SMD:C_0805_2012Metric_Pad1.18x1.45mm_HandSolder
- C9: renamed from C6; footprint (none) -> Capacitor_SMD:C_0805_2012Metric_Pad1.18x1.45mm_HandSolder
- D3, D4: footprint (none) -> LED_SMD:LED_0805_2012Metric_Pad1.15x1.40mm_HandSolder
- J6: renamed from J3; footprint (none) -> 0_AKeller_Footprints:USB_Micro-B_Amphenol
- U2: renamed from U3; footprint Package_SO:SSOP-28_5.3x10.2mm_P0.65mm -> 0_AKeller_Footprints:SSOP-28
Connections:
- net RX: now also TP1.1
- net TX: now also TP2.1
- net at C11.1, J6.3 (D+), U2.15 (USBD+): now also TP3.1
- net at C10.1, J6.2 (D-), U2.16 (USBD-): now also TP4.1

Commit message: Master board silkscreen and gerber files
Other:
- title: UART -> Laser Arcade Master
Changed lines of the file:
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@@
 	(paper "A")
 	(title_block
-		(title "UART")
-		(date "2025-04-04")
+		(title "Laser Arcade Master")
+		(date "2025-04-17")
 		(rev "A")
 		(company "Idaho State University")
