File: KiCad/Target_Slave/Target_Slave.kicad_pcb (KiCad board)
At the start: 2 copper layers, 76.2 x 50.8 mm, 36 parts, among them J1 ICSP, J2 I2C, J3 I2C, SW1 I2C Address, U1 PIC16F1788-IP, U2 TSSP4038, U3 TSOP53456

Commit message: Add Silkscreen text, Add logos
Parts:
- added G***: LOGO, 2025 Logos:RCET Stacked 1x_33, F.Cu at (189.9, 88.3)
- added G***: LOGO, 2025 Logos:Benny _5x_5, B.Cu at (229.2, 108.0)
- added G***: LOGO, 2025 Logos:AKeller_Logo_0-4x0-3, B.Cu at (175.9, 118.1)
Routing:
- net Net-(D2-RK): track 94.0 -> 95.2 mm
Other:
- board text added: "+5V"
- board text added: "GND"
- board text added: "Laser Arcade Target Slave Rev. A Spring 2025"
- board text added: "SCL"
- board text added: "SDA"

Commit message: Master PCB design, Slave board logos
Parts:
- added TP1: ~, 0_AKeller_Footprints:1x1_100mil_Header, F.Cu at (208.3, 99.7)
- added TP2: ~, 0_AKeller_Footprints:1x1_100mil_Header, F.Cu at (181.6, 108.0)
- added TP3: ~, 0_AKeller_Footprints:1x1_100mil_Header, F.Cu at (181.6, 102.9)
- added TP4: ~, 0_AKeller_Footprints:1x1_100mil_Header, F.Cu at (198.1, 99.7)
Routing:
- net Net-(U1-RC3/SCK/SCL): track 137.9 -> 151.6 mm
- net Net-(U1-P1C/AN10/RB1): track 10.5 -> 13.3 mm
- net Net-(U1-INT/AN12/RB0): track 9.24 -> 12.1 mm
- net GND: track 46.0 -> 48.7 mm
- net Net-(U1-RC4/SDI/SDA): track 134.5 -> 133.8 mm

Commit message: Slave Gerbers
Parts:
- added G***: LOGO, 2025 Logos:Alex_Logo, B.Cu at (186.7, 123.4)
- moved D2 0.76 mm to (188.0, 96.5)
- moved D3 0.23 mm to (223.5, 96.5)
Routing:
- net Net-(D2-BK): track 93.3 -> 92.1 mm
- net Net-(D2-RK): track 95.2 -> 95.8 mm
Other:
- board text added: "D2"
- board text added: "D3"
- board text added: "D4"
- board text added: "D5"
