File: KiCad/Target_Slave/Target_Slave.kicad_sch (KiCad schematic)
At the start: 36 parts, among them J1 ICSP, J2 I2C, J3 I2C, SW1 I2C Address, U1 PIC16F1788-IP, U2 TSSP4038, U3 TSOP53456

Commit message: Target Slave Revision B schematic update
Parts:
- removed C4: 1uF, Capacitor_SMD:C_0805_2012Metric_Pad1.18x1.45mm_HandSolder, symbol Device:C_Small
- removed D2, D3, D4, D5: IN-P32TRRRGB, 0_AKeller_Footprints:IN-P32TRRRGB, symbol Libraries:RGB_LED_P32TRRRGB
- removed R1, R2, R3, R4, R5, R6, R7, R8: 330Ω, Resistor_SMD:R_0805_2012Metric_Pad1.20x1.40mm_HandSolder, symbol Libraries:R_Custom
- removed R10, R12: 90Ω, Resistor_SMD:R_0805_2012Metric_Pad1.20x1.40mm_HandSolder, symbol Libraries:R_Custom
- removed R11: 150Ω, Resistor_SMD:R_0805_2012Metric_Pad1.20x1.40mm_HandSolder, symbol Libraries:R_Custom
- removed R13: 4.7kΩ, Resistor_SMD:R_0805_2012Metric_Pad1.20x1.40mm_HandSolder, symbol Libraries:R_Custom
- removed R9: 10kΩ, Resistor_SMD:R_0805_2012Metric_Pad1.20x1.40mm_HandSolder, symbol Libraries:R_Custom
- removed SW1: I2C Address, 0_AKeller_Footprints:SW_DIP_SPSTx08_Slide_9.78x22.5mm_W7.62mm_P2.54mm, symbol Switch:SW_DIP_x08
- removed U3: TSOP53456, 0_AKeller_Footprints:IR Receiver, symbol Interface_Optical:TSOP331xx
- added D2: WS2812B, LED_SMD:LED_WS2812B_PLCC4_5.0x5.0mm_P3.2mm, symbol LED:WS2812B
- added D3: Hit Indicator, LED_SMD:LED_0805_2012Metric_Pad1.15x1.40mm_HandSolder, symbol Device:LED_Filled
- added J2: LED, symbol 0_AKeller_Parts:Header_1x3
- added JP1: Mode, symbol Jumper:Jumper_3_Bridged12
- added R1: 10kΩ, symbol Device:R_US
- added R2: 470Ω, symbol Device:R_US
- added R3, R4: 4.7kΩ, symbol Device:R_US
- added TP1, TP10, TP2, TP3, TP8, TP9: ~, 0_AKeller_Footprints:1x1_100mil_Header, symbol 0_AKeller_Parts:Test_Point
- D4: renamed from D6; value LED -> Power
- renumbered C5 to C4, C6 to C5, J2 to J3, J3 to J4, TP2 to TP5, TP3 to TP6, TP1 to TP7
Connections:
- net +5V: now also D2.1 (VDD), J2.1, R1.1, TP10.1
- net GND: now also D2.3 (VSS), J2.2, R3.2, R4.2
- net at D1.1 (K), J1.1, U1.1 (RE3/~{MCLR}/Vpp): now also TP1.1
- net at TP7.1, U2.1 (OUT): now also JP1.1 (A); no longer U1.21 (INT/AN12/RB0)
- net at U1.22 (P1C/AN10/RB1): no longer TP4.1
- net at D4.1 (K): now also R4.1
- net at C2.1, D1.2 (A): now also R1.2
- net RA0: no longer names the net of U1.2 (ULPWU/C12IN0-/AN0/RA0)
- net RA0: now also R2.1, TP2.1
- net RA1: no longer names the net of U1.3 (C12IN1-/AN1/RA1)
- net RA1: now also TP4.1, D3.2 (A)
- net RA2: no longer names the net of U1.4 (CVref/C2IN1+/Vref-/AN2/RA2)
- net RA3: no longer names the net of U1.5 (C1IN+/Vref+/AN3/RA3)
- net RA4: no longer names the net of U1.6 (T0CKI/C1OUT/RA4)
- net RA5: no longer names the net of U1.7 (~{SS}/C2OUT/AN4/RA5)
- net RA6: no longer names the net of U1.10 (CLKOUT/OSC2/RA6)
- net RA7: no longer names the net of U1.9 (CLKIN/OSC1/RA7)
- net RB6 renamed TX
- net TX: now also TP8.1
- net RB7: no longer names the net of U1.28 (ICSPDAT/RB7)
- net RB7: now also JP1.2 (C); no longer J1.4
- new net: D3.1 (K), R3.1
- new net: D2.2 (DOUT), J2.3, TP3.1
- new net: D2.4 (DIN), R2.2
- new net RX: J1.4, JP1.3 (B), TP9.1
- no-connect marks 8 -> 19
Other:
- note added: "1 - 5V 2 - GND 3 - SIG"
- note added: "Game"
- note added: "Program"
- note removed: "56kHz IR Receiever"
- note removed: "In-Circuit Serial Programming"
- moved on the sheet: C3, TP7, U2
