File: KiCad/Project.kicad_pcb (KiCad board)
At the start: 2 copper layers, 129.7 x 40.6 mm, 53 parts, among them J2 Power & Output Test Points, J3 Inputs Test Points, Q1 BUK9832-55A, Q2 BUK9832-55A, Q3 BUK9832-55A, SW1 Power, SW2 Fire, SW3 Freq Select, SW4 Fire Select, U1 TLV1117-50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

Commit message: finished blaster PCB
Parts:
- added G***: LOGO, LOGO, F.Cu at (177.6, 79.7)
- added G***: LOGO, LOGO, F.Cu at (165.8, 90.3)
- added G***: LOGO, LOGO, F.Cu at (94.7, 89.5)
- added G***: LOGO, LOGO, B.Cu at (83.4, 101.3)
- added G***: LOGO, LOGO, B.Cu at (77.9, 88.0)
- added G***: LOGO, LOGO, B.Cu at (177.4, 81.4)
- added G***: LOGO, LOGO, B.Cu at (190.0, 95.1)
- moved ? 61.1 mm to (135.7, 112.6)
- moved ? 61.1 mm to (135.7, 79.6)
- moved C1 61.1 mm to (196.8, 93.8)
- moved C3 61.1 mm to (192.7, 87.2)
- moved C4 61.1 mm to (185.0, 79.3)
- moved C6 61.1 mm to (140.1, 90.8)
- moved D1 61.1 mm to (191.4, 96.6)
- moved D3 61.1 mm to (191.4, 93.9)
- moved J1 61.1 mm to (152.7, 114.4)
- moved Q1 61.1 mm to (157.7, 98.7)
- moved Q3 61.1 mm to (171.6, 98.7)
- moved R1 61.1 mm to (184.8, 96.6)
- moved R10 61.1 mm to (152.4, 100.8)
- moved R11 61.1 mm to (166.3, 100.8)
- moved R12 61.1 mm to (152.4, 102.8)
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Connections:
- U2 pad 19: Net-(U2-VSS-Pad19) -> GND
- U2 pad 2: unconnected-(U2-ULPWU/C12IN0-/AN0/RA0-Pad2) -> TRIG0
- U2 pad 8: Net-(U2-VSS-Pad19) -> GND
Routing:
- net GND: track 52.6 -> 239.0 mm, vias 2 -> 12
- net +5V_Top: track 97.7 -> 123.6 mm
- net Net-(Q3-G): track 99.2 -> 87.3 mm
- net Net-(Q1-G): track 42.0 -> 51.6 mm
- net Solenoid: track 19.3 -> 25.9 mm
- net Laser/PWM: track 6.53 -> 12.8 mm
- net Laser/PWM2: track 6.05 -> 12.4 mm
- net +5V: track 170.1 -> 176.0 mm
- net RB7: track 77.1 -> 82.4 mm
- net Net-(U2-VSS-Pad19): track 3.86 -> 0.00 mm
- net Net-(Q2-S): track 0.07 -> 2.29 mm
- net TRIG6: track 20.1 -> 19.2 mm
- net Net-(Q2-G): track 44.6 -> 43.8 mm
- net RB6: track 38.2 -> 38.8 mm
- net Full-Auto_Top: track 44.9 -> 44.3 mm
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Other:
- board text added: "GitHub"
- board text added: "ICSP"
- board text added: "Laser Arcade Blaster (Bottom) Rev. A Alex Wheelock Spring 2025"
- board text added: "Laser Arcade Blaster (Top) Rev. A Alex Wheelock Spring 2025"
- board text added: "Laser1"
- board text added: "Solenoid"
- board text removed: "Program"
