File: KiCad/Blaster_Power.kicad_sch (KiCad schematic)
At the start: 12 parts, among them SW1 Power, U1 TLV1117-50

Commit message: updated blaster schematic
Parts:
- BT1: value 7.4V -> +12V
Connections:
- net +7.4V_Top renamed +12V_Top
Changed lines of the file:
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@@
 		)
 	)
-	(global_label "+7.4V_Top"
+	(global_label "+12V_Top"
 		(shape output)
 		(at 81.28 78.74 0)
@@
 		)
 		(property "Intersheetrefs" "${INTERSHEET_REFS}"
-			(at 94.1832 78.74 0)
+			(at 93.5784 78.74 0)
 			(effects
 				(font
@@
 			)
 		)
-		(property "Value" "+7.4V"
+		(property "Value" "+12V"
 			(at 127 78.74 0)
 			(effects
@@
 			)
 		)
-		(property "Value" "7.4V"
+		(property "Value" "+12V"
 			(at 63.5 88.3284 0)
 			(effects
